File: Hardware/VL6180_Sensor.brd (EAGLE design)
At the start: 44.5 x 13 mm, 25 parts, among them Q1 BSS138, Q2 BSS138, U1 VL6180, U3 MIC5219 3.3V

Commit message: Updating VL6180 library path
Parts:
- U1: device VL6180:VL6180 -> SparkFun-Sensors:VL6180
